File: PCB/lamp_ceiling/lamp_ceiling/lamp_ceiling.kicad_pcb (KiCad board)
At the start: 2 copper layers, 55 parts, among them J1 LED_supply, J10 LED_supply, J11 LED1_NTC, J12 LED1_fan, J13 LED_supply, J14 LED1_NTC, J15 LED1_fan, J2 LED1_NTC, J3 LED1_fan, J4 LED_supply, J5 LED1_NTC, J6 LED1_fan, J7 LED_supply, J8 LED1_NTC, J9 LED1_fan, Q1 DMG1012UW-7, Q10 DMG1012UW-7, Q2 DMG1012UW-7, Q3 DMG1012UW-7, Q4 DMG1012UW-7, Q5 DMG1012UW-7, Q6 DMG1012UW-7, Q7 DMG1012UW-7, Q8 DMG1012UW-7, Q9 DMG1012UW-7, U1 LMV321IDBVR, U2 LMV321IDBVR, U3 LMV321IDBVR, U4 LMV321IDBVR, U5 MCP3208, U6 LMV321IDBVR, U7 MIC5504-3.3YM5, U9 STM32F030R8Tx

Commit message: started layout
Parts:
- added C1: 100nF, Capacitor_SMD:C_0603_1608Metric, F.Cu at (102.8, 65.8)
- added C11: 100nF, Capacitor_SMD:C_0603_1608Metric, F.Cu at (135.8, 103.0)
- added C2: 100nF, Capacitor_SMD:C_0603_1608Metric, F.Cu at (102.8, 90.7)
- added C3: 100nF, Capacitor_SMD:C_0603_1608Metric, F.Cu at (102.8, 115.5)
- added C4: 100nF, Capacitor_SMD:C_0603_1608Metric, F.Cu at (96.0, 128.0)
- added R10: 20k, 1%, Resistor_SMD:R_0603_1608Metric, F.Cu at (96.0, 69.2)
- added R11: 20k, 1%, Resistor_SMD:R_0603_1608Metric, F.Cu at (96.0, 91.2)
- added R12: 20k, 1%, Resistor_SMD:R_0603_1608Metric, F.Cu at (96.0, 94.2)
- added R13: 20k, 1%, Resistor_SMD:R_0603_1608Metric, F.Cu at (96.0, 116.0)
- added R14: 20k, 1%, Resistor_SMD:R_0603_1608Metric, F.Cu at (96.0, 119.0)
- added R15: 20k, 1%, Resistor_SMD:R_0603_1608Metric, F.Cu at (87.2, 131.8)
- added R16: 20k, 1%, Resistor_SMD:R_0603_1608Metric, F.Cu at (90.2, 131.8)
- added R17: 100k, 1%, Resistor_SMD:R_0603_1608Metric, F.Cu at (99.5, 70.5)
- added R18: 100k, 1%, Resistor_SMD:R_0603_1608Metric, F.Cu at (99.7, 95.5)
- added R19: 100k, 1%, Resistor_SMD:R_0603_1608Metric, F.Cu at (99.8, 120.2)
- added R20: 100k, 1%, Resistor_SMD:R_0603_1608Metric, F.Cu at (93.0, 132.6)
- added R21: 100k, 1%, Resistor_SMD:R_0603_1608Metric, F.Cu at (99.5, 65.0)
- added R22: 100k, 1%, Resistor_SMD:R_0603_1608Metric, F.Cu at (99.5, 90.0)
- added R23: 100k, 1%, Resistor_SMD:R_0603_1608Metric, F.Cu at (99.5, 114.8)
- added R24: 100k, 1%, Resistor_SMD:R_0603_1608Metric, F.Cu at (93.0, 127.2)
- added R27: 20k, 1%, Resistor_SMD:R_0603_1608Metric, F.Cu at (144.8, 104.5)
- added R28: 20k, 1%, Resistor_SMD:R_0603_1608Metric, F.Cu at (141.8, 107.5)
- added R29: 100k, 1%, Resistor_SMD:R_0603_1608Metric, F.Cu at (136.0, 130.2)
- added R31: 100k, 1%, Resistor_SMD:R_0603_1608Metric, F.Cu at (144.8, 107.5)
- added R9: 20k, 1%, Resistor_SMD:R_0603_1608Metric, F.Cu at (96.0, 66.2)
- moved R4 101.7 mm to (88.8, 134.8), turned to 180 degrees
- moved J10 98.4 mm to (83.2, 141.8), turned to 90 degrees
- moved Q8 98.3 mm to (88.0, 138.0), turned to 270 degrees
- moved R8 96.0 mm to (92.8, 134.8), turned to 180 degrees
- moved J11 96.0 mm to (90.2, 141.8), turned to 90 degrees
- moved Q3 89.5 mm to (87.4, 127.4), turned to 180 degrees
- moved J12 89.1 mm to (97.2, 141.8), turned to 90 degrees
- moved J14 87.4 mm to (115.2, 141.8), turned to 90 degrees
- moved J8 86.8 mm to (83.2, 123.8)
- moved J7 85.2 mm to (83.2, 116.8)
- moved Q5 78.7 mm to (88.0, 67.0), turned to 180 degrees
- moved U3 77.8 mm to (99.8, 117.5)
- moved J9 77.7 mm to (83.2, 130.7)
- moved J13 75.3 mm to (108.2, 141.8), turned to 90 degrees
- moved R26 75.2 mm to (113.2, 132.8), turned to 180 degrees
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Connections:
- Q5 pad 1: LED1_PWM -> (no net)
- Q7 pad 1: LED1_PWM -> (no net)
- Q8 pad 1: LED1_PWM -> (no net)
- U1 pad 1: (no net) -> Net-(R21-Pad1)
- U1 pad 3: (no net) -> Net-(R10-Pad2)
- U2 pad 1: (no net) -> Net-(R11-Pad2)
- U2 pad 3: (no net) -> Net-(R12-Pad2)
- U3 pad 1: (no net) -> Net-(R13-Pad2)
- U3 pad 3: (no net) -> Net-(R14-Pad2)
- U4 pad 1: (no net) -> Net-(R15-Pad2)
- U4 pad 3: (no net) -> Net-(R16-Pad2)
- U6 pad 1: (no net) -> Net-(R27-Pad2)
- U6 pad 3: (no net) -> Net-(R28-Pad2)
